Commit message: Feat: added extra simulation properties - launch file to start simulation - paths added to cmakelists -  needed dependencies added to package.xml - world file need to be fixed, i will handle it - some xacro macros edited to fix path problems (to add meshes with using package keyword)

File: auv_description/models/prototype_vehicle/macros/pipe_macro.xacro (robot description, xacro)
@@ -2,5 +2,5 @@
 <robot xmlns:xacro="http://www.ros.org/wiki/xacro">
   <xacro:macro name="add_pipe" params="name length x y z r p yaw radius:=0.0125">
-    <visual name="${name}_visual">
+    <!-- <visual name="${name}_visual">
       <origin xyz="${x} ${y} ${z}" rpy="${r} ${p} ${yaw}"/>
       <geometry>
@@ -10,5 +10,5 @@
         <color rgba="0.1 0.1 0.1 1"/>
       </material>
-    </visual>
+    </visual> -->
     <collision name="${name}_collision">
       <origin xyz="${x} ${y} ${z}" rpy="${r} ${p} ${yaw}"/>

File: auv_description/models/prototype_vehicle/macros/plugins.xacro (robot description, xacro)
@@ -29,4 +29,7 @@
       <control channel="7"><jointName>thruster8_joint</jointName><servo_min>1100</servo_min><servo_max>1900</servo_max><type>COMMAND</type><cmd_topic>/model/prototype/joint/thruster8_joint/cmd_thrust</cmd_topic><offset>-0.5</offset><multiplier>100</multiplier></control>
     </plugin>
+        <plugin filename="gz-sim-joint-state-publisher-system" name="gz::sim::systems::JointStatePublisher">
+      <update_rate>50</update_rate>
+      <topic>/model/prototype_vehicle/joint_state</topic> </plugin>
   </gazebo>
 </robot>

File: auv_description/models/prototype_vehicle/macros/thruster_macro.xacro (robot description, xacro)
@@ -6,5 +6,5 @@
         <origin xyz="0 0 0" rpy="-1.571 0 0"/>
         <geometry>
-          <mesh filename="model://bluerov2_heavy/meshes/t200_${prop_type}_prop.dae"/>
+          <mesh filename="package://auv_description/models/bluerov2_heavy/meshes/t200_${prop_type}_prop.dae"/>
         </geometry>
       </visual>

File: auv_description/models/prototype_vehicle/prototype.urdf (robot description, URDF)
Before this commit: robot prototype, 9 links, 8 joints
Links:
- link base_link: mass 11.0 -> 5.0; geometry collision cylinder length=0.0702 radius=0.0125; collision cylinder length=0.0702 radius=0.0125
- link thruster1: geometry visual mesh filename=package://auv_description/models/bluerov2_heavy/meshes/t200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
- link thruster2: geometry visual mesh filename=package://auv_description/models/bluerov2_heavy/meshes/t200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
- link thruster3: geometry visual mesh filename=package://auv_description/models/bluerov2_heavy/meshes/t200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
- link thruster4: geometry visual mesh filename=package://auv_description/models/bluerov2_heavy/meshes/t200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
- link thruster5: geometry visual mesh filename=package://auv_description/models/bluerov2_heavy/meshes/t200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
- link thruster6: geometry visual mesh filename=package://auv_description/models/bluerov2_heavy/meshes/t200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
- link thruster7: geometry visual mesh filename=package://auv_description/models/bluerov2_heavy/meshes/t200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
- link thruster8: geometry visual mesh filename=package://auv_description/models/bluerov2_heavy/meshes/t200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
Joints:
- joint thruster1_joint: type continuous -> revolute
- joint thruster2_joint: type continuous -> revolute
- joint thruster3_joint: type continuous -> revolute
- joint thruster4_joint: type continuous -> revolute
- joint thruster5_joint: type continuous -> revolute
- joint thruster6_joint: type continuous -> revolute
- joint thruster7_joint: type continuous -> revolute
- joint thruster8_joint: type continuous -> revolute

File: auv_description/models/prototype_vehicle/prototype.urdf.xacro (robot description, xacro)
@@ -8,9 +8,9 @@
     <inertial>
       <origin xyz="0 0 -0.05" rpy="0 0 0"/>
-      <mass value="11.0"/>
+      <mass value="10.0"/>
       <inertia ixx="0.201" ixy="0" ixz="0" iyy="0.223" iyz="0" izz="0.269"/>
     </inertial>
     <visual>
-      <geometry><mesh filename="model://prototype_vehicle/meshes/sim.obj"/></geometry>
+      <geometry><mesh filename="package://auv_description/models/prototype_vehicle/meshes/sim.obj"/></geometry>
     </visual>
     <xacro:add_pipe name="left_top_pipe"   length="0.365"  x="0.001"  y="0.156"   z="0.1417" r="0" p="${pi/2}" yaw="0" />
