Commit message: Fix: buoyancy problem fixed - it was sinking or jumping regardless of the mass, to fix that i checked the bluerov2 model and I used the method which they use to define collisions and visuals - There was a problem because of center of mass, vehicle wasnt stable, i allocated center of mass at the z axis to the : -0.06 - spawning point changed - hydrodinamics parameters(added masses, and linear quadratic damping things will be adjusted when Nehir calculate)

File: auv_description/models/prototype_vehicle/macros/plugins.xacro (robot description, xacro)
@@ -5,10 +5,22 @@
       <link_name>base_link</link_name>
       <water_density>1000.0</water_density>
-      <xDotU>0</xDotU> <yDotV>0</yDotV> <zDotW>0</zDotW>
-      <kDotP>0</kDotP> <mDotQ>0</mDotQ> <nDotR>0</nDotR>
-      <xU>0</xU> <yV>0</yV> <zW>0</zW>
-      <kP>0</kP> <mQ>0</mQ> <nR>0</nR>
-      <xUabsU>-58.42</xUabsU> <yVabsV>-55.137</yVabsV> <zWabsW>-124.818</zWabsW>
-      <kPabsP>-4.0</kPabsP>   <mQabsQ>-4.0</mQabsQ>   <nRabsR>-4.0</nRabsR>
+      <xDotU>5.0</xDotU>
+      <yDotV>5.0</yDotV>
+      <zDotW>5.0</zDotW>
+      <kDotP>0</kDotP>
+      <mDotQ>0</mDotQ>
+      <nDotR>0</nDotR>
+      <xU>-20.0</xU>
+      <yV>-20.0</yV>
+      <zW>-20.0</zW>
+      <kP>-10.0</kP>
+      <mQ>-10.0</mQ>
+      <nR>-10.0</nR>
+      <xUabsU>-17.1</xUabsU>
+      <yVabsV>-25.65</yVabsV>
+      <zWabsW>-27.0</zWabsW>
+      <kPabsP>-4.0</kPabsP>
+      <mQabsQ>-4.0</mQabsQ>
+      <nRabsR>-4.0</nRabsR>
     </plugin>
     <plugin name="ArduPilotPlugin" filename="libArduPilotPlugin.so">
@@ -29,7 +41,13 @@
       <control channel="7"><jointName>thruster8_joint</jointName><servo_min>1100</servo_min><servo_max>1900</servo_max><type>COMMAND</type><cmd_topic>/model/prototype/joint/thruster8_joint/cmd_thrust</cmd_topic><offset>-0.5</offset><multiplier>100</multiplier></control>
     </plugin>
-        <plugin filename="gz-sim-joint-state-publisher-system" name="gz::sim::systems::JointStatePublisher">
+    <plugin filename="gz-sim-joint-state-publisher-system" name="gz::sim::systems::JointStatePublisher">
       <update_rate>50</update_rate>
-      <topic>/model/prototype_vehicle/joint_state</topic> </plugin>
+      <topic>/model/prototype_vehicle/joint_state</topic>
+    </plugin>
+    <plugin filename="gz-sim-odometry-publisher-system" name="gz::sim::systems::OdometryPublisher">
+      <odom_frame>odom</odom_frame>
+      <robot_base_frame>base_link</robot_base_frame>
+      <dimensions>3</dimensions>
+    </plugin>
   </gazebo>
 </robot>

File: auv_description/models/prototype_vehicle/prototype.urdf.xacro (robot description, xacro)
@@ -7,37 +7,27 @@
   <link name="base_link">
     <inertial>
-      <origin xyz="0 0 -0.05" rpy="0 0 0"/>
-      <mass value="2.0"/>
-      <inertia ixx="0.201" ixy="0" ixz="0" iyy="0.223" iyz="0" izz="0.269"/>
+      <origin xyz="0 0 -0.06" rpy="0 0 0"/>
+      <mass value="10.5"/>
+      <inertia
+          ixx="0.073" ixy="0" ixz="0"
+          iyy="0.121" iyz="0"
+          izz="0.125"/>
     </inertial>
     <visual>
-      <geometry><mesh filename="package://auv_description/models/prototype_vehicle/meshes/sim.obj"/></geometry>
+      <origin xyz="0 0 0" rpy="0 0 0"/>
+      <geometry>
+        <mesh filename="package://auv_description/models/prototype_vehicle/meshes/sim.obj"/>
+      </geometry>
     </visual>
-    <xacro:add_pipe name="left_top_pipe"   length="0.365"  x="0.001"  y="0.156"   z="0.1417" r="0" p="${pi/2}" yaw="0" />
-    <xacro:add_pipe name="right_top_pipe"  length="0.365"  x="0.001"  y="-0.156"  z="0.1417" r="0" p="${pi/2}" yaw="0" />
-    <xacro:add_pipe name="back_top_pipe"   length="0.3354" x="-0.182" y="-0.0017" z="0.1413" r="${pi/2}" p="0" yaw="0" />
-    <xacro:add_pipe name="front_top_pipe"  length="0.3354" x="0.182"  y="-0.0017" z="0.1413" r="${pi/2}" p="0" yaw="0" />
-    <xacro:add_pipe name="left_bottom_pipe"  length="0.365"  x="0.001"  y="0.156"   z="-0.123" r="0" p="${pi/2}" yaw="0" />
-    <xacro:add_pipe name="right_bottom_pipe" length="0.365"  x="0.001"  y="-0.156"  z="-0.123" r="0" p="${pi/2}" yaw="0" />
-    <xacro:add_pipe name="back_bottom_pipe"  length="0.3354" x="-0.182" y="-0.0017" z="-0.123" r="${pi/2}" p="0" yaw="0" />
-    <xacro:add_pipe name="front_bottom_pipe" length="0.3354" x="0.182"  y="-0.0017" z="-0.123" r="${pi/2}" p="0" yaw="0" />
-    <xacro:add_pipe name="front_left_pipe"  length="0.25" x="0.1857"  y="-0.0760" z="0.01" r="0" p="0" yaw="0" />
-    <xacro:add_pipe name="front_right_pipe" length="0.25" x="0.1857"  y="0.0760"  z="0.01" r="0" p="0" yaw="0" />
-    <xacro:add_pipe name="back_right_pipe"  length="0.25" x="-0.1857" y="0.0760"  z="0.01" r="0" p="0" yaw="0" />
-    <xacro:add_pipe name="back_left_pipe"   length="0.25" x="-0.1857" y="-0.0760" z="0.01" r="0" p="0" yaw="0" />
-    <xacro:add_pipe name="inner_front_left_pipe"   length="0.25" x="0.1057" y="0.1690" z="0.01" r="0" p="0" yaw="0" />
-    <xacro:add_pipe name="inner_front_right_pipe"   length="0.25" x="0.1057" y="-0.1690" z="0.01" r="0" p="0" yaw="0" />
-    <xacro:add_pipe name="inner_back_left_pipe"   length="0.25" x="-0.1057" y="0.1690" z="0.01" r="0" p="0" yaw="0" />
-    <xacro:add_pipe name="inner_back_right_pipe"   length="0.25" x="-0.1057" y="-0.1690" z="0.01" r="0" p="0" yaw="0" />
-    <xacro:add_pipe name="left_mid_back_horizontal_pipe" length="0.0702" x="-0.1058" y="0.1140" z="0.0198" r="${pi/2}" p="0" yaw="0" />
-    <xacro:add_pipe name="left_mid_front_horizontal_pipe" length="0.0702" x="0.1058" y="0.1140" z="0.0198" r="${pi/2}" p="0" yaw="0" />
-    <xacro:add_pipe name="right_mid_front_horizontal_pipe" length="0.0702" x="0.1058" y="-0.1140" z="0.0198" r="${pi/2}" p="0" yaw="0" />
-    <xacro:add_pipe name="right_mid_back_horizontal_pipe" length="0.0702" x="-0.1058" y="-0.1140" z="0.0198" r="${pi/2}" p="0" yaw="0" />
-    <xacro:add_pipe name="left_mid_long_pipe" length="0.33" x="0.0007" y="0.0744" z="0.02" r="0" p="${pi/2}" yaw="0" />
-    <xacro:add_pipe name="right_mid_long_pipe" length="0.33" x="0.0007" y="-0.0744" z="0.02" r="0" p="${pi/2}" yaw="0" />
-    <xacro:add_pipe name="enclosure" length="0.35" radius="0.055" x="0.0007" y="-0.001" z="0.01" r="0" p="${pi/2}" yaw="0" />
-</link>
-  <xacro:add_imu name="imu_sensor" parent_link="base_link" update_rate="400.0" x="0" y="0" z="0" r="${pi}" p="0" yaw="0" />
-  <xacro:add_imu name="vio_imu" parent_link="base_link" update_rate="300.0" topic="/imu0" x="0" y="0" z="0" r="0" p="0" yaw="0" />
+    <collision name="base_collision">
+      <geometry>
+        <box size="0.30 0.20 0.19"/>
+      </geometry>
+    </collision>
+  </link>
+  <xacro:add_imu name="imu_sensor" parent_link="base_link" update_rate="400.0"
+                 x="0" y="0" z="0" r="${pi}" p="0" yaw="0" />
+  <xacro:add_imu name="vio_imu" parent_link="base_link" update_rate="300.0" topic="/imu0"
+                 x="0" y="0" z="0" r="0" p="0" yaw="0" />
   <xacro:add_thruster id="1" x="0.2201"  y="-0.1126" z="-0.0224" r="-1.571" p="1.571" yaw="-0.785" prop_type="ccw" coeff="0.02" />
   <xacro:add_thruster id="2" x="0.2201"  y="0.1126"  z="-0.0224" r="-1.571" p="1.571" yaw="-2.356" prop_type="ccw" coeff="0.02" />
