Commit message: Fix: last changes done

File: auv_description/models/prototype_vehicle/macros/camera_macro.xacro (robot description, xacro)
@@ -17,6 +17,6 @@
       </collision>
       <inertial>
-        <mass value="0.1"/>
-        <inertia ixx="0.00016" ixy="0" ixz="0" iyy="0.00016" iyz="0" izz="0.00016"/>
+        <mass value="0.00000001"/>
+        <inertia ixx="0.00000001" ixy="0" ixz="0" iyy="0.00000001" iyz="0" izz="0.00000001"/>
       </inertial>
     </link>

File: auv_description/models/prototype_vehicle/macros/plugins.xacro (robot description, xacro)
@@ -5,19 +5,11 @@
       <link_name>base_link</link_name>
       <water_density>1000.0</water_density>
-      <xDotU>5.0</xDotU>
-      <yDotV>5.0</yDotV>
-      <zDotW>5.0</zDotW>
-      <kDotP>0</kDotP>
-      <mDotQ>0</mDotQ>
-      <nDotR>0</nDotR>
-      <xU>-20.0</xU>
-      <yV>-20.0</yV>
-      <zW>-20.0</zW>
-      <kP>-10.0</kP>
-      <mQ>-10.0</mQ>
-      <nR>-10.0</nR>
-      <xUabsU>-17.1</xUabsU>
-      <yVabsV>-55.3</yVabsV>
-      <zWabsW>-55.0</zWabsW>
+      <xDotU>0</xDotU> <yDotV>0</yDotV> <zDotW>0</zDotW>
+      <kDotP>0</kDotP> <mDotQ>0</mDotQ> <nDotR>0</nDotR>
+      <xU>-5.0</xU> <yV>-5.0</yV> <zW>-5.0</zW>
+      <kP>-5.0</kP> <mQ>-5.0</mQ> <nR>-5.0</nR>
+      <xUabsU>-58.42</xUabsU>
+      <yVabsV>-55.137</yVabsV>
+      <zWabsW>-124.818</zWabsW>
       <kPabsP>-4.0</kPabsP>
       <mQabsQ>-4.0</mQabsQ>
@@ -32,5 +24,5 @@
       <gazeboXYZToNED>0 0 0 3.142 0 1.571</gazeboXYZToNED>
       <imuName>imu_sensor</imuName>
-      <control channel="0"><jointName>thruster1_joint</jointName><servo_min>1000</servo_min><servo_max>2000</servo_max><type>COMMAND</type><cmd_topic>/model/prototype_vehicle/joint/thruster1_joint/cmd_thrust</cmd_topic><offset>-0.5</offset><multiplier>100</multiplier></control>
+      <control channel="0"><jointName>thruster1_joint</jointName><servo_min>1100</servo_min><servo_max>1900</servo_max><type>COMMAND</type><cmd_topic>/model/prototype_vehicle/joint/thruster1_joint/cmd_thrust</cmd_topic><offset>-0.5</offset><multiplier>100</multiplier></control>
       <control channel="1"><jointName>thruster2_joint</jointName><servo_min>1100</servo_min><servo_max>1900</servo_max><type>COMMAND</type><cmd_topic>/model/prototype_vehicle/joint/thruster2_joint/cmd_thrust</cmd_topic><offset>-0.5</offset><multiplier>100</multiplier></control>
       <control channel="2"><jointName>thruster3_joint</jointName><servo_min>1100</servo_min><servo_max>1900</servo_max><type>COMMAND</type><cmd_topic>/model/prototype_vehicle/joint/thruster3_joint/cmd_thrust</cmd_topic><offset>-0.5</offset><multiplier>100</multiplier></control>

File: auv_description/models/prototype_vehicle/macros/sonar_macro.xacro (robot description, xacro)
@@ -7,6 +7,6 @@
     <link name="${name}_link">
       <inertial>
-        <mass value="0.05"/> <origin xyz="0 0 0" rpy="0 0 0"/>
-        <inertia ixx="0.0001" ixy="0" ixz="0" iyy="0.0001" iyz="0" izz="0.0001"/>
+        <mass value="0.00000001"/> <origin xyz="0 0 0" rpy="0 0 0"/>
+        <inertia ixx="0.00000001" ixy="0" ixz="0" iyy="0.00000001" iyz="0" izz="0.00000001"/>
       </inertial>
       <visual>

File: auv_description/models/prototype_vehicle/prototype.urdf.xacro (robot description, xacro)
@@ -9,10 +9,9 @@
   <link name="base_link">
     <inertial>
-      <origin xyz="0 0 -0.06" rpy="0 0 0"/>
-      <mass value="10.5"/>
-      <inertia
-          ixx="0.073" ixy="0" ixz="0"
-          iyy="0.121" iyz="0"
-          izz="0.125"/>
+      <origin xyz="0 0 -0.0114" rpy="0 0 0"/>
+      <mass value="12.8"/> <inertia
+        ixx="0.26" ixy="0" ixz="0"
+        iyy="0.23" iyz="0"
+        izz="0.37"/>
     </inertial>
     <visual>
@@ -23,6 +22,7 @@
     </visual>
     <collision name="base_collision">
+      <origin xyz="0 0 0.376" rpy="0 0 0"/>
       <geometry>
-        <box size="0.30 0.20 0.19"/>
+        <box size="0.457 0.575 0.05"/>
       </geometry>
     </collision>
@@ -42,5 +42,5 @@
     parent_link="base_link"
     topic="/camera/front"
-    x="0.178062" y="0.0" z="0.0"
+    x="0.177035" y="0.0" z="0.0"
     r="0.0" p="0.0" yaw="0.0"
     color="Blue" />
@@ -62,5 +62,5 @@
   <xacro:add_thruster id="2" x="0.2201"  y="0.1126"  z="-0.0224" r="-1.571" p="1.571" yaw="-2.356" prop_type="ccw" coeff="0.02" />
   <xacro:add_thruster id="3" x="-0.2201" y="-0.1126" z="-0.0224" r="-1.571" p="1.571" yaw="0.785"  prop_type="cw"  coeff="-0.02" />
-  <xacro:add_thruster id="4" x="-0.2201" y="0.1126"  z="-0.0224" r="-1.571" p="1.571" yaw="0.785"  prop_type="cw"  coeff="-0.02" />
+  <xacro:add_thruster id="4" x="-0.2201" y="0.1126"  z="-0.0224" r="-1.571" p="1.571" yaw="2.356"  prop_type="cw"  coeff="-0.02" />
   <xacro:add_thruster id="5" x="0.0884"  y="-0.2126" z="0.0056"  r="0" p="0" yaw="0" prop_type="ccw" coeff="0.02" />
   <xacro:add_thruster id="6" x="0.0884"  y="0.2126"  z="0.0056"  r="0" p="0" yaw="0" prop_type="cw"  coeff="-0.02" />
