Commit message: Fix centre of buoyancy, camera intrinsics, and sensor frame ids
Four real defects found while auditing the sim against Gazebo Harmonic
(gz-sensors 8), which is what sim_dvl_bridge.py's gz.transport13/gz.msgs10
imports pin us to.

1. base_link's buoyancy collision sat at z=0.376, 20cm above the hull's
   actual top (the visual mesh ends at z=0.145) - a dropped zero. That put
   the centre of buoyancy 0.387m above the CoM instead of 0.049m, an 8x too
   stiff righting moment (48.6 vs 6.2 N*m/rad) and a vehicle that could
   never float up to the surface. 0.0376 reproduces exactly the 0.049m
   CoB-CoM separation that bluerov2_heavy/model.sdf uses for the same hull.
   NOTE: this genuinely changes roll/pitch dynamics - re-check mission tuning.

2. Nothing ever published /camera/camera_info, so bbox_pnp_solver blocked
   forever on intrinsics and never solved a single pose: gz derives the
   camera_info topic from the scoped sensor path unless told otherwise. Set
   <camera_info_topic> per camera (<image topic>/camera_info), bridge all
   three, and point yolo.launch.py + the node default at the front camera's,
   which is the camera yolo_node actually reads.

3. Revert my earlier frame_id change back to gz_frame_id. gz-sensors 8 reads
   ONLY gz_frame_id (src/Sensor.cc); frame_id lands in gz-sensors 9 (Ionic),
   which then deprecates gz_frame_id. On Harmonic my frame_id was silently
   ignored, leaving the sensors with auto-generated scoped frames. Comment
   added so the next person swaps it on the Ionic upgrade instead of
   "fixing" it back.

4. Drop two bridge entries that could never carry data
   (/world/deneme/dynamic_pose/info - wrong world name and the world is gone;
   /model/prototype_vehicle/pose - no PosePublisher plugin exists) and give
   the flight IMU an explicit topic so its entry resolves. ArduPilotPlugin
   binds that IMU by sensor name, not topic, so it is unaffected.

Also: cameras 100 -> 30 Hz and the Ping1D 30 -> 10 Hz. Three 640x480 render
passes at 100 Hz is more than the GPU delivers, so the sim was paying real
time factor for frames it never produced; both rates now match the hardware.

Co-Authored-By: Claude Opus 5 <noreply@anthropic.com>

File: auv_description/models/prototype_vehicle/macros/camera_macro.xacro (robot description, xacro)
@@ -30,6 +30,13 @@
       <sensor name="${name}" type="camera">
         <pose>0 0 0 0 0 0</pose>
-        <frame_id>${name}_link</frame_id>
+        <!-- gz_frame_id, not frame_id: see the note in ping1d_macro.xacro. -->
+        <gz_frame_id>${name}_link</gz_frame_id>
         <camera>
+          <!-- Publish intrinsics next to the image (<topic>/camera_info).
+               Without this gz still derives a camera_info topic, but from the
+               fully-scoped sensor path, which is not what the vision nodes
+               subscribe to - bbox_pnp_solver sat waiting on a topic that
+               never existed. Keep this in sync with bridge.yaml. -->
+          <camera_info_topic>${topic}/camera_info</camera_info_topic>
           <horizontal_fov>1.047</horizontal_fov> <!-- 60 Derece -->
           <image>
@@ -59,5 +66,9 @@
         </camera>
         <always_on>true</always_on>
-        <update_rate>100</update_rate>
+        <!-- 30 Hz, matching the real cameras. Was 100: three 640x480 render
+             passes at 100 Hz is far more than the GPU delivers, so the sim
+             just loses real-time factor while the images still arrive late
+             and irregularly. Nothing downstream consumes faster than 30. -->
+        <update_rate>30</update_rate>
         <visualize>true</visualize>
         <topic>${topic}</topic>

File: auv_description/models/prototype_vehicle/macros/dvl_macro.xacro (robot description, xacro)
@@ -38,5 +38,6 @@
         <update_rate>${update_rate}</update_rate>
         <always_on>true</always_on>
-        <frame_id>${name}_link</frame_id>
+        <!-- gz_frame_id, not frame_id: see the note in ping1d_macro.xacro. -->
+        <gz_frame_id>${name}_link</gz_frame_id>
         <gz:dvl>
           <type>phased_array</type>

File: auv_description/models/prototype_vehicle/macros/ping1d_macro.xacro (robot description, xacro)
@@ -38,8 +38,13 @@
         <pose>0 0 0 0 0 0</pose>
         <topic>${topic}</topic>
-        <update_rate>30</update_rate>
+        <!-- Real Ping1D pings at roughly 10 Hz; it is time-of-flight bound,
+             it cannot do 30. Also one fewer GPU render pass per frame. -->
+        <update_rate>10</update_rate>
         <always_on>true</always_on>
         <visualize>true</visualize>
-        <frame_id>${name}_link</frame_id>
+        <!-- gz_frame_id, NOT frame_id: gz-sensors 8 (Harmonic, what this repo
+             targets) only reads gz_frame_id. frame_id arrives in gz-sensors 9
+             (Ionic), which then deprecates this one - swap on that upgrade. -->
+        <gz_frame_id>${name}_link</gz_frame_id>
         <lidar>
           <scan>

File: auv_description/models/prototype_vehicle/prototype.urdf.xacro (robot description, xacro)
@@ -22,6 +22,14 @@
       </geometry>
     </visual>
+    <!-- This box is what the world's Buoyancy plugin displaces, so its VOLUME
+         sets net buoyancy (0.457*0.575*0.05 * 1000 = 13.14 kg vs 12.8 kg mass,
+         i.e. slightly positive) and its CENTROID is the centre of buoyancy.
+         z=0.0376 puts the CoB 0.049 m above the CoM at z=-0.0114 - the same
+         separation bluerov2_heavy/model.sdf uses (0.060 vs 0.011).
+         Was 0.376 (a dropped zero): that sat 20 cm above the hull's actual
+         top (the mesh ends at z=0.145), giving an 8x too stiff righting
+         moment and a vehicle that could never float to the surface. -->
     <collision name="base_collision">
-      <origin xyz="0 0 0.376" rpy="0 0 0"/>
+      <origin xyz="0 0 0.0376" rpy="0 0 0"/>
       <geometry>
         <box size="0.457 0.575 0.05"/>
@@ -29,5 +37,10 @@
     </collision>
   </link>
+  <!-- Flight IMU. ArduPilotPlugin binds to it by sensor NAME (<imuName>), not
+       by topic; the explicit topic is only so bridge.yaml can expose it to ROS
+       for debugging. Without it gz publishes on the fully-scoped sensor path
+       and the bridge entry matches nothing. -->
   <xacro:add_imu name="imu_sensor" parent_link="base_link" update_rate="400.0"
+                 topic="/model/prototype_vehicle/imu"
                  x="0" y="0" z="0" r="${pi}" p="0" yaw="0" />
   <xacro:add_imu name="vio_imu" parent_link="base_link" update_rate="50.0" topic="/imu0"
