Commit message: feat: torpedo launcher added and some little changes on torpedo's inertia

File: auv_description/models/prototype_vehicle/macros/torpedo.xacro (robot description, xacro)
@@ -3,5 +3,5 @@
   <link name="torpedo_body">
     <inertial>
-      <mass value="0.3"/>
+      <mass value="0.05"/>
       <origin xyz="0 0 0" rpy="0 1.5708 0"/>
       <inertia ixx="0.001" iyy="0.001" izz="0.001" ixy="0" ixz="0" iyz="0"/>
@@ -19,5 +19,5 @@
       <origin xyz="0 0 0" rpy="0 1.5708 0"/>
       <geometry>
-        <cylinder radius="0.03" length="0.2"/>
+        <cylinder radius="0.04" length="0.2"/>
       </geometry>
     </collision>

Commit message: feat: double torpedo launch mechanism added

File: auv_description/models/prototype_vehicle/macros/torpedo.xacro (robot description, xacro)
@@ -1,4 +1,5 @@
 <?xml version="1.0"?>
 <robot xmlns:xacro="http://www.ros.org/wiki/xacro" name="torpedo_model">
+  <xacro:arg name="torp_id" default="1"/>
   <link name="torpedo_body">
     <inertial>
@@ -9,16 +10,10 @@
     <visual>
       <origin xyz="0 0 0" rpy="0 1.5708 0"/>
-      <geometry>
-        <cylinder radius="0.03" length="0.2"/>
-      </geometry>
-      <material name="orange">
-        <color rgba="1.0 0.5 0.0 1.0"/>
-      </material>
+      <geometry><cylinder radius="0.03" length="0.2"/></geometry>
+      <material name="orange"><color rgba="1.0 0.5 0.0 1.0"/></material>
     </visual>
     <collision>
       <origin xyz="0 0 0" rpy="0 1.5708 0"/>
-      <geometry>
-        <cylinder radius="0.04" length="0.2"/>
-      </geometry>
+      <geometry><cylinder radius="0.04" length="0.2"/></geometry>
     </collision>
   </link>
@@ -35,15 +30,6 @@
     <axis xyz="1 0 0"/>
   </joint>
-  <gazebo reference="torpedo_body">
-    <visual>
-      <material>
-        <ambient>1.0 0.0 0.0 1.0</ambient> <diffuse>1.0 0.0 0.0 1.0</diffuse>
-        <specular>0.1 0.1 0.1 1.0</specular>
-      </material>
-    </visual>
-  </gazebo>
 <gazebo>
     <plugin filename="gz-sim-thruster-system" name="gz::sim::systems::Thruster">
-      <namespace>torpedo</namespace>
       <joint_name>propeller_joint</joint_name>
       <thrust_coefficient>0.01</thrust_coefficient>
@@ -51,5 +37,5 @@
       <propeller_diameter>0.05</propeller_diameter>
       <velocity_control>true</velocity_control>
-      <topic>/torpedo/cmd_thrust</topic>
+      <topic>/torpedo/cmd_thrust$(arg torp_id)</topic>
     </plugin>
   </gazebo>

File: auv_description/models/prototype_vehicle/prototype.urdf.xacro (robot description, xacro)
@@ -74,7 +74,15 @@
     <plugin filename="gz-sim-detachable-joint-system" name="gz::sim::systems::DetachableJoint">
       <parent_link>base_link</parent_link>
-      <child_model>torpedo_model</child_model>
+      <child_model>torpedo_model1</child_model>
       <child_link>torpedo_body</child_link>
-      <detach_topic>/torpedo/fire</detach_topic>
+      <detach_topic>/torpedo/fire1</detach_topic>
+    </plugin>
+  </gazebo>
+    <gazebo>
+    <plugin filename="gz-sim-detachable-joint-system" name="gz::sim::systems::DetachableJoint">
+      <parent_link>base_link</parent_link>
+      <child_model>torpedo_model2</child_model>
+      <child_link>torpedo_body</child_link>
+      <detach_topic>/torpedo/fire2</detach_topic>
     </plugin>
   </gazebo>
