Commit message: Textured pool model, dedupe worlds, real Ping1D + DVL sensors
- New auv_description/models/pool: 25x50m competition pool as a reusable
  model (5x5m tiled PBR floor + walls), textures ported from
  HonuRobotics/bluerobotics_models (Apache-2.0, see NOTICE). Replaces the
  ~200 lines of hand-placed, flat-colored floor/wall SDF that used to live
  inline in teknofest_pool.world with a single <include>.
- Remove deneme.world, pool.world, underwater.world: none were referenced
  by any launch file; only teknofest_pool.world and open_water.world are
  actually used.
- sonar_macro.xacro -> ping1d_macro.xacro: wire up the Ping1D sonar that
  was sitting commented out in prototype.urdf.xacro, tune range to the
  real datasheet (0.5-50m), fix the topic (was missing the leading slash
  bridge.yaml expects) and swap the non-standard <gz_frame_id> tag for the
  real <frame_id> so the sensor's TF frame actually resolves.
- dvl_macro.xacro: give the DVL a visible body (it had a sensor with no
  link at all before) and correct <type> from piston to phased_array to
  match the real Water Linked DVL-A50 and the ROS-side bridge, which
  already mapped that type and only ever received the wrong one. Renamed
  the vehicle's DVL instance to "dvl" so its frame_id ("dvl_link") matches
  what sim_dvl_bridge.py/sim_dvl_adapter.py already assume.
- auv_description/README.md: rewrite to match what's actually in the
  package (it described a urdf/ dir and launch files that don't exist).

Co-Authored-By: Claude Sonnet 5 <noreply@anthropic.com>

File: auv_description/models/prototype_vehicle/macros/dvl_macro.xacro (robot description, xacro)
@@ -1,13 +1,44 @@
 <?xml version="1.0"?>
+<!-- Water Linked DVL-A50 macro. Real hardware is a phased-array (electronic
+beam steering) transducer, not a mechanical piston, and the driver referenced
+by this repo (additional_drivers/waterlinked_dvl) targets that same A50. -->
 <robot xmlns:xacro="http://www.ros.org/wiki/xacro" xmlns:gz="http://gazebosim.org/schema">
   <xacro:macro name="add_dvl" params="name parent_link topic update_rate x y z r p yaw">
-    <gazebo reference="${parent_link}">
+    <link name="${name}_link">
+      <inertial>
+        <mass value="0.00000001"/> <origin xyz="0 0 0" rpy="0 0 0"/>
+        <inertia ixx="0.00000001" ixy="0" ixz="0" iyy="0.00000001" iyz="0" izz="0.00000001"/>
+      </inertial>
+      <!-- DVL-A50: 73.5mm diameter, ~40mm tall puck. -->
+      <visual>
+        <origin xyz="0 0 0" rpy="0 0 0"/>
+        <geometry>
+          <cylinder length="0.04" radius="0.0368"/>
+        </geometry>
+        <material name="dvl_black">
+          <color rgba="0.08 0.08 0.08 1"/>
+        </material>
+      </visual>
+      <collision>
+        <origin xyz="0 0 0" rpy="0 0 0"/>
+        <geometry>
+          <cylinder length="0.04" radius="0.0368"/>
+        </geometry>
+      </collision>
+    </link>
+    <joint name="${name}_joint" type="fixed">
+      <parent link="${parent_link}"/>
+      <child link="${name}_link"/>
+      <origin xyz="${x} ${y} ${z}" rpy="${r} ${p} ${yaw}"/>
+    </joint>
+    <gazebo reference="${name}_link">
       <sensor name="${name}" type="custom" gz:type="dvl">
-        <pose>${x} ${y} ${z} ${r} ${p} ${yaw}</pose>
+        <pose>0 0 0 0 0 0</pose>
         <topic>${topic}</topic>
         <update_rate>${update_rate}</update_rate>
         <always_on>true</always_on>
+        <frame_id>${name}_link</frame_id>
         <gz:dvl>
-          <type>piston</type>
+          <type>phased_array</type>
           <arrangement degrees="true">
             <beam id="1">

File: auv_description/models/prototype_vehicle/macros/ping1d_macro.xacro (robot description, xacro)
@@ -1,8 +1,12 @@
 <?xml version="1.0"?>
-<!-- SONAR MACRO FILE (to import simulation), we are using gazebo's lidar sensor to imitate bluerobotics' sonar 1D
-a cone created, which apical angle is approximately 30 degree (as like blue sonar),
-and the parameters can be adjusted depending intended usage case -->
+<!-- Blue Robotics Ping1D (Ping Sonar Altimeter/Echosounder) macro.
+gz-sim has no dedicated single-beam sonar sensor, so this imitates the
+Ping1D with a narrow gpu_lidar: a ~30 deg apical cone (matching the Ping1D
+datasheet beam width) sampled at 32x32 rays instead of the single physical
+transducer's one range reading. A consumer that wants the real Ping1D
+behaviour (one Range message) should reduce this scan to its minimum valid
+return, not consume every ray as if it were a multi-beam sonar. -->
 <robot xmlns:xacro="http://www.ros.org/wiki/xacro">
-  <xacro:macro name="add_sonar" params="name parent_link topic x y z r p yaw">
+  <xacro:macro name="add_ping1d" params="name parent_link topic x y z r p yaw">
     <link name="${name}_link">
       <inertial>
@@ -37,5 +41,5 @@
         <always_on>true</always_on>
         <visualize>true</visualize>
-        <gz_frame_id>${name}_link</gz_frame_id>
+        <frame_id>${name}_link</frame_id>
         <lidar>
           <scan>
@@ -48,6 +52,6 @@
           </scan>
           <range>
-            <min>0.2</min>
-            <max>30.0</max> <resolution>0.01</resolution>
+            <min>0.5</min>
+            <max>50.0</max> <resolution>0.01</resolution>
           </range>
           <noise>

File: auv_description/models/prototype_vehicle/prototype.urdf.xacro (robot description, xacro)
@@ -5,5 +5,5 @@
   <xacro:include filename="macros/plugins.xacro" />
   <xacro:include filename="macros/imu_macro.xacro"/>
-  <xacro:include filename="macros/sonar_macro.xacro" />
+  <xacro:include filename="macros/ping1d_macro.xacro" />
   <xacro:include filename="macros/camera_macro.xacro" />
   <xacro:include filename="macros/dvl_macro.xacro" />
@@ -33,11 +33,10 @@
   <xacro:add_imu name="vio_imu" parent_link="base_link" update_rate="50.0" topic="/imu0"
                  x="0" y="0" z="0" r="0" p="0" yaw="0" />
-<!--
-  <xacro:add_sonar
-      name="ping_sonar"
+  <xacro:add_ping1d
+      name="ping1d_sonar"
       parent_link="base_link"
-      topic="sensors/sonar/front"
+      topic="/sensors/sonar/front"
       x="0.188254" y="-0.038661" z="0.09952"
-      r="0.0" p="0.0" yaw="0.0" /> -->
+      r="0.0" p="0.0" yaw="0.0" />
   <xacro:add_camera
     name="front_camera"
@@ -62,5 +61,5 @@
     color="Green" />
   <xacro:add_dvl
-    name="dvl_sensor"
+    name="dvl"
     parent_link="base_link"
     topic="/model/prototype_vehicle/dvl"
