Commit message: Fix: World file path errors fixed - used ament env hooks to solve path errors (it could not find sand_heightmap model and AI suggested that)

File: auv_description/models/prototype_vehicle/prototype.urdf.xacro (robot description, xacro)
@@ -8,5 +8,5 @@
     <inertial>
       <origin xyz="0 0 -0.05" rpy="0 0 0"/>
-      <mass value="10.0"/>
+      <mass value="2.0"/>
       <inertia ixx="0.201" ixy="0" ixz="0" iyy="0.223" iyz="0" izz="0.269"/>
     </inertial>
